File: 16-key.kicad_pcb (KiCad board)
At the start: 2 copper layers, 34 parts, among them U1 ProMicro

Commit message: basically done
Parts:
- added MICROSD1: PINHD-1X8LOCK, Connector_PinHeader_1.00mm:PinHeader_1x08_P1.00mm_Vertical, F.Cu at (173.8, 85.7)
- moved RESET1 7.94 mm to (184.2, 58.7)
- moved U1 7.94 mm to (183.4, 38.9)
Connections:
- U1 pad 14: Net-(U1-Pad14) -> DI
- U1 pad 15: Net-(U1-Pad15) -> DO
- U1 pad 16: Net-(U1-Pad16) -> CLK
- U1 pad 17: Net-(U1-Pad17) -> CS
- U1 pad 18: Net-(U1-Pad18) -> CO
Routing:
- net COL0: track 0.00 -> 187.3 mm
- net COL1: track 0.00 -> 175.2 mm
- net COL2: track 0.00 -> 148.6 mm
- net ROW3: track 0.00 -> 113.9 mm
- net ROW2: track 0.00 -> 97.4 mm
- net COL3: track 0.00 -> 85.4 mm
- net ROW1: track 0.00 -> 80.1 mm
- net GND: track 0.00 -> 76.2 mm
- net ROW0: track 0.00 -> 72.3 mm
- net CO: track 0.00 -> 56.0 mm
- net +5V: track 0.00 -> 53.3 mm
- net CS: track 0.00 -> 51.7 mm
- net CLK: track 0.00 -> 43.9 mm
- net DO: track 0.00 -> 42.4 mm
- net DI: track 0.00 -> 40.9 mm
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Other:
- board outline added: 113.5 x 81 mm
- board text added: "16-Key"
- board text added: "Future Micro SD Card Board"
- board text added: "clw 2020-01-09 Rev. A"

Commit message: added pull up resistor
Parts:
- added R1: 100k, Resistor_SMD:R_0805_2012Metric, F.Cu at (182.4, 55.6)
Routing:
- net Net-(R1-Pad1): track 30.3 -> 33.8 mm
- net +5V: track 53.3 -> 55.0 mm

Commit message: moved lettering to silk screen
Other:
- board text added: "JLCJLCJLCJLC"
Changed lines of the file:
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@@
   (general
     (thickness 1.6)
-    (drawings 11)
+    (drawings 12)
     (tracks 108)
     (zones 0)
@@
     (visible_elements FFFFFF7F)
     (pcbplotparams
-      (layerselection 0x010fc_ffffffff)
-      (usegerberextensions false)
-      (usegerberattributes true)
+      (layerselection 0x010f0_ffffffff)
+      (usegerberextensions true)
+      (usegerberattributes false)
       (usegerberadvancedattributes true)
-      (creategerberjobfile true)
+      (creategerberjobfile false)
       (excludeedgelayer true)
       (linewidth 0.100000)
@@
       (outputformat 1)
       (mirror false)
-      (drillshape 1)
+      (drillshape 0)
       (scaleselection 1)
-      (outputdirectory ""))
+      (outputdirectory "Gerbers/"))
   )
   (net 0 "")
@@
     (fp_line (start 1.68 -0.95) (end 1.68 0.95) (layer F.CrtYd) (width 0.05))
     (fp_line (start 1.68 0.95) (end -1.68 0.95) (layer F.CrtYd) (width 0.05))
-    (pad 2 smd roundrect (at 0.9125 0 180) (size 1.025 1.4) (layers F.Cu F.Paste F.Mask) (roundrect_rratio 0.243902)
+    (pad 2 smd roundrect (at 0.9125 0 180) (size 1.025 1.4) (layers F.Cu F.Paste F.Mask) (roundrect_rratio 0.2439014634146341)
       (net 35 +5V))
-    (pad 1 smd roundrect (at -0.9125 0 180) (size 1.025 1.4) (layers F.Cu F.Paste F.Mask) (roundrect_rratio 0.243902)
+    (pad 1 smd roundrect (at -0.9125 0 180) (size 1.025 1.4) (layers F.Cu F.Paste F.Mask) (roundrect_rratio 0.2439014634146341)
       (net 47 "Net-(R1-Pad1)"))
     (model ${KISYS3DMOD}/Resistor_SMD.3dshapes/R_0805_2012Metric.wrl
@@
     )
   )
-  (gr_text "clw 2020-01-09 Rev. A" (at 184.15 100.80625) (layer Dwgs.User)
+  (gr_text "Future Micro SD Card Board" (at 185.7375 82.55) (layer F.SilkS)
     (effects (font (size 1 1) (thickness 0.15)))
   )
-  (gr_text "Future Micro SD Card Board" (at 186.53125 82.55) (layer Dwgs.User)
+  (gr_text 16-Key (at 171.45 97.63125) (layer F.SilkS)
     (effects (font (size 1 1) (thickness 0.15)))
   )
-  (gr_text 16-Key (at 171.45 99.21875) (layer Dwgs.User)
+  (gr_text "clw 2020-01-09 Rev. A" (at 184.94375 100.0125) (layer F.SilkS)
     (effects (font (size 1 1) (thickness 0.15)))
   )
+  (gr_text JLCJLCJLCJLC (at 189.70625 92.86875) (layer B.SilkS)
+    (effects (font (size 1 1) (thickness 0.15)) (justify mirror))
+  )
   (gr_line (start 197.64375 26.19375) (end 197.64375 96.8375) (layer Edge.Cuts) (width 0.05))

Commit message: added mounting holes
Parts:
- added ?: , Connector_Pin:Pin_D1.0mm_L10.0mm, F.Cu at (180.2, 92.9)
- added ?: , Connector_Pin:Pin_D1.0mm_L10.0mm, F.Cu at (169.1, 29.4)
- added ?: , Connector_Pin:Pin_D1.0mm_L10.0mm, F.Cu at (88.9, 26.2)
- added ?: , Connector_Pin:Pin_D1.0mm_L10.0mm, F.Cu at (88.9, 97.6)
Changed lines of the file:
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@@
     (tracks 108)
     (zones 0)
-    (modules 36)
+    (modules 40)
     (nets 48)
   )
@@
     (add_net ROW3)
   )
+  (module Connector_Pin:Pin_D1.0mm_L10.0mm (layer F.Cu)
+    (at 180.18125 92.86875)
+    (descr "solder Pin_ diameter 1.0mm, hole diameter 1.0mm (press fit), length 10.0mm")
+    (tags "solder Pin_ press fit")
+    (fp_text reference "" (at 0 2.25) (layer F.SilkS) hide
+      (effects (font (size 1 1) (thickness 0.15)))
+    )
+    (fp_text value "" (at 0 -2.05) (layer F.Fab)
+      (effects (font (size 10 10) (thickness 0.15)))
+    )
+    (fp_circle (center 0 0) (end 1.5 0) (layer F.CrtYd) (width 0.05))
+    (fp_circle (center 0 0) (end 0.5 0) (layer F.Fab) (width 0.12))
+    (fp_circle (center 0 0) (end 1 0) (layer F.Fab) (width 0.12))
+    (fp_circle (center 0 0) (end 1.25 0.05) (layer F.SilkS) (width 0.12))
+    (fp_text user %R (at 0 2.25) (layer F.Fab)
+      (effects (font (size 10 10) (thickness 0.15)))
+    )
+    (pad "" thru_hole circle (at 0 0) (size 4.2 4.2) (drill 3.2) (layers *.Cu *.Mask))
+    (model ${KISYS3DMOD}/Connector_Pin.3dshapes/Pin_D1.0mm_L10.0mm.wrl
+      (at (xyz 0 0 0))
+      (scale (xyz 1 1 1))
+      (rotate (xyz 0 0 0))
+    )
+  )
+  (module Connector_Pin:Pin_D1.0mm_L10.0mm (layer F.Cu)
+    (at 169.06875 29.36875)
+    (descr "solder Pin_ diameter 1.0mm, hole diameter 1.0mm (press fit), length 10.0mm")
+    (tags "solder Pin_ press fit")
+    (fp_text reference "" (at 0 2.25) (layer F.SilkS) hide
+      (effects (font (size 1 1) (thickness 0.15)))
+    )
+    (fp_text value "" (at 0 -2.05) (layer F.Fab)
+      (effects (font (size 10 10) (thickness 0.15)))
+    )
+    (fp_circle (center 0 0) (end 1.5 0) (layer F.CrtYd) (width 0.05))
+    (fp_circle (center 0 0) (end 0.5 0) (layer F.Fab) (width 0.12))
+    (fp_circle (center 0 0) (end 1 0) (layer F.Fab) (width 0.12))
+    (fp_circle (center 0 0) (end 1.25 0.05) (layer F.SilkS) (width 0.12))
+    (fp_text user %R (at 0 2.25) (layer F.Fab)
+      (effects (font (size 10 10) (thickness 0.15)))
+    )
+    (pad "" thru_hole circle (at 0 0) (size 4.2 4.2) (drill 3.2) (layers *.Cu *.Mask))
+    (model ${KISYS3DMOD}/Connector_Pin.3dshapes/Pin_D1.0mm_L10.0mm.wrl
+      (at (xyz 0 0 0))
+      (scale (xyz 1 1 1))
+      (rotate (xyz 0 0 0))
+    )
+  )
+  (module Connector_Pin:Pin_D1.0mm_L10.0mm (layer F.Cu)
+    (at 88.9 26.19375)
+    (descr "solder Pin_ diameter 1.0mm, hole diameter 1.0mm (press fit), length 10.0mm")
+    (tags "solder Pin_ press fit")
+    (fp_text reference "" (at 0 2.25) (layer F.SilkS) hide
+      (effects (font (size 1 1) (thickness 0.15)))
+    )
+    (fp_text value "" (at 0 -2.05) (layer F.Fab)
+      (effects (font (size 10 10) (thickness 0.15)))
+    )
+    (fp_circle (center 0 0) (end 1.5 0) (layer F.CrtYd) (width 0.05))
+    (fp_circle (center 0 0) (end 0.5 0) (layer F.Fab) (width 0.12))
+    (fp_circle (center 0 0) (end 1 0) (layer F.Fab) (width 0.12))
+    (fp_circle (center 0 0) (end 1.25 0.05) (layer F.SilkS) (width 0.12))
+    (fp_text user %R (at 0 2.25) (layer F.Fab)
+      (effects (font (size 10 10) (thickness 0.15)))
+    )
+    (pad "" thru_hole circle (at 0 0) (size 4.2 4.2) (drill 3.2) (layers *.Cu *.Mask))
+    (model ${KISYS3DMOD}/Connector_Pin.3dshapes/Pin_D1.0mm_L10.0mm.wrl
+      (at (xyz 0 0 0))
+      (scale (xyz 1 1 1))
+      (rotate (xyz 0 0 0))
+    )
+  )
+  (module Connector_Pin:Pin_D1.0mm_L10.0mm (layer F.Cu)
+    (at 88.9 97.63125)
+    (descr "solder Pin_ diameter 1.0mm, hole diameter 1.0mm (press fit), length 10.0mm")
+    (tags "solder Pin_ press fit")
+    (fp_text reference "" (at 0 2.25) (layer F.SilkS) hide
+      (effects (font (size 1 1) (thickness 0.15)))
+    )
+    (fp_text value "" (at 0 -2.05) (layer F.Fab)
+      (effects (font (size 10 10) (thickness 0.15)))
+    )
+    (fp_text user %R (at 0 2.25) (layer F.Fab)
+      (effects (font (size 10 10) (thickness 0.15)))
+    )
+    (fp_circle (center 0 0) (end 1.5 0) (layer F.CrtYd) (width 0.05))
+    (fp_circle (center 0 0) (end 0.5 0) (layer F.Fab) (width 0.12))
+    (fp_circle (center 0 0) (end 1 0) (layer F.Fab) (width 0.12))
+    (fp_circle (center 0 0) (end 1.25 0.05) (layer F.SilkS) (width 0.12))
+    (pad "" thru_hole circle (at 0 0) (size 4.2 4.2) (drill 3.2) (layers *.Cu *.Mask))
+    (model ${KISYS3DMOD}/Connector_Pin.3dshapes/Pin_D1.0mm_L10.0mm.wrl
+      (at (xyz 0 0 0))
+      (scale (xyz 1 1 1))
+      (rotate (xyz 0 0 0))
+    )
+  )
   (module Resistor_SMD:R_0805_2012Metric (layer F.Cu)
